File: 24S_Counter.kicad_pcb (KiCad board)
At the start: 2 copper layers, 0 parts

Commit message: final commit
Parts:
- added G***: LOGO, LOGO, F.Cu at (88.5, 131.0)
- added H1: MountingHole, MountingHole:MountingHole_2.2mm_M2, F.Cu at (81.0, 79.5)
- added H2: MountingHole, MountingHole:MountingHole_2.2mm_M2, F.Cu at (150.5, 79.5)
- added H3: MountingHole, MountingHole:MountingHole_2.2mm_M2, F.Cu at (150.5, 132.0)
- added H4: MountingHole, MountingHole:MountingHole_2.2mm_M2, F.Cu at (80.5, 131.5)
- added J1: +5V, my_footprints:Terminal_Block_5mm, F.Cu at (90.5, 80.0)
- added J2: EXT_CLK, Connector_PinHeader_2.54mm:PinHeader_1x02_P2.54mm_Vertical, F.Cu at (87.5, 118.3)
- added R1: 100R, Resistor_SMD:R_1206_3216Metric_Pad1.30x1.75mm_HandSolder, F.Cu at (114.0, 91.5)
- added R10: 100R, Resistor_SMD:R_1206_3216Metric_Pad1.30x1.75mm_HandSolder, F.Cu at (145.2, 123.3)
- added R11: 100R, Resistor_SMD:R_1206_3216Metric_Pad1.30x1.75mm_HandSolder, F.Cu at (145.2, 127.3)
- added R12: 100R, Resistor_SMD:R_1206_3216Metric_Pad1.30x1.75mm_HandSolder, F.Cu at (145.1, 131.3)
- added R13: 100R, Resistor_SMD:R_1206_3216Metric_Pad1.30x1.75mm_HandSolder, F.Cu at (140.4, 86.5)
- added R14: 100R, Resistor_SMD:R_1206_3216Metric_Pad1.30x1.75mm_HandSolder, F.Cu at (134.5, 86.5)
- added R15: 1K, Resistor_SMD:R_1206_3216Metric_Pad1.30x1.75mm_HandSolder, F.Cu at (109.0, 127.0)
- added R16: 10K, Resistor_SMD:R_1206_3216Metric_Pad1.30x1.75mm_HandSolder, F.Cu at (109.0, 122.5)
- added R17: 1K, Resistor_SMD:R_1206_3216Metric_Pad1.30x1.75mm_HandSolder, F.Cu at (92.5, 123.0)
- added R18: 10K, Resistor_SMD:R_1206_3216Metric_Pad1.30x1.75mm_HandSolder, F.Cu at (92.5, 116.5)
- added R2: 100R, Resistor_SMD:R_1206_3216Metric_Pad1.30x1.75mm_HandSolder, F.Cu at (114.0, 95.5)
- added R3: 100R, Resistor_SMD:R_1206_3216Metric_Pad1.30x1.75mm_HandSolder, F.Cu at (114.0, 99.5)
- added R4: 100R, Resistor_SMD:R_1206_3216Metric_Pad1.30x1.75mm_HandSolder, F.Cu at (114.0, 103.5)
- added R5: 100R, Resistor_SMD:R_1206_3216Metric_Pad1.30x1.75mm_HandSolder, F.Cu at (114.0, 107.0)
- added R6: 100R, Resistor_SMD:R_1206_3216Metric_Pad1.30x1.75mm_HandSolder, F.Cu at (122.5, 86.0)
- added R7: 100R, Resistor_SMD:R_1206_3216Metric_Pad1.30x1.75mm_HandSolder, F.Cu at (114.0, 88.0)
- added R8: 100R, Resistor_SMD:R_1206_3216Metric_Pad1.30x1.75mm_HandSolder, F.Cu at (145.1, 115.3)
- added R9: 100R, Resistor_SMD:R_1206_3216Metric_Pad1.30x1.75mm_HandSolder, F.Cu at (145.1, 119.3)
- added SW1: EN, my_footprints:slide_switch_2.54mm, F.Cu at (99.0, 119.5)
- added SW2: RST, my_footprints:tact_switch_5mm, F.Cu at (109.0, 117.0)
- added U1: 74LS192, my_footprints:74LS192, F.Cu at (90.3, 98.8)
- added U2: 74LS192, my_footprints:74LS192, F.Cu at (121.1, 122.8)
- added U3: 74LS48, my_footprints:74LS48, F.Cu at (102.8, 99.0)
- added U4: 74LS48, my_footprints:74LS48, F.Cu at (134.3, 122.7)
- added U5: SM420561N, Display_7Segment:7SegmentLED_LTS6760_LTS6780, F.Cu at (121.4, 106.6)
- added U6: SM420561N, Display_7Segment:7SegmentLED_LTS6760_LTS6780, F.Cu at (136.4, 106.6)
Routing:
- net GND: track 0.00 -> 194.0 mm
- net /+5V: track 0.00 -> 147.4 mm, vias 0 -> 3
- net /B0: track 0.00 -> 61.2 mm
- net /Load: track 0.00 -> 59.0 mm, vias 0 -> 1
- net Net-(U1-QC): track 0.00 -> 39.4 mm
- net Net-(U4-f): track 0.00 -> 38.8 mm
- net Net-(U6-E): track 0.00 -> 38.3 mm, vias 0 -> 1
- net Net-(U2-QC): track 0.00 -> 36.3 mm
- net Net-(U4-g): track 0.00 -> 34.5 mm
- net Net-(U6-B): track 0.00 -> 32.9 mm, vias 0 -> 1
- net Net-(U1-QD): track 0.00 -> 30.5 mm, vias 0 -> 1
- net Net-(U1-QA): track 0.00 -> 30.3 mm
- net /CLK: track 0.00 -> 28.6 mm, vias 0 -> 1
- net Net-(U2-QD): track 0.00 -> 28.4 mm, vias 0 -> 1
- net Net-(U6-A): track 0.00 -> 28.2 mm, vias 0 -> 1
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Other:
- board outline added: 77.5 x 62.5 mm
- board text added: "24 SECOND COUNTER"
- board text added: "Design Engineer: Cid Lawrenc Regalado Dare: 13 Apr 2026"
